Commit message: fix status

File: floor/floor_description/urdf/floor.urdf (robot description, URDF)
Before this commit: robot floor, 6 links, 5 joints
Joints:
- joint joint1: limit lower=-0.26 upper=0.26 effort=1000 velocity=1.5 -> lower=-0.52 upper=0.52 effort=1000 velocity=1.5
- joint joint2: limit lower=-0.26 upper=0.26 effort=1000 velocity=1.5 -> lower=-0.52 upper=0.52 effort=1000 velocity=1.5

File: floor/floor_description/urdf/floor.urdf.xacro (robot description, xacro)
@@ -11,5 +11,5 @@
   <xacro:property name="height4" value="0.05" /> <!-- Link 4 -->
   <xacro:property name="width4" value="2" /> <!-- Link 4 -->
-  <xacro:property name="limit_joint" value="0.26" /> <!-- Limit joint-->
+  <xacro:property name="limit_joint" value="0.52" /> <!-- Limit joint-->
   <xacro:property name="camera_link" value="0.05" /> <!-- Size of square 'camera' box -->
   <xacro:property name="axel_offset" value="0.05" /> <!-- Space btw top of beam and the each joint -->
