Commit message: ready to train

File: floor/floor_description/urdf/floor.urdf.xacro (robot description, xacro)
@@ -120,4 +120,12 @@
     <origin xyz="0 0 ${height3}" rpy="0 0 0"/>
   </joint>
+      <!-- <surface>
+        <friction>
+          <ode>
+            <mu>1</mu>
+            <mu2>1</mu2>
+          </ode>
+        </friction>
+      </surface> -->
     <!-- Base Link -->
   <link name="link4">
@@ -144,4 +152,13 @@
     </inertial>
   </link>
+  <gazebo reference="link4">
+    <kp>1000000.0</kp>
+    <kd>1.0</kd>
+    <mu1>0.9</mu1>
+    <mu2>0.9</mu2>
+    <maxVel>0.0</maxVel>
+    <minDepth>0.001</minDepth>
+    <material>Gazebo/Orange</material>
+  </gazebo>
   <link name="imu_link">
     <inertial>

File: oped/oped_description/urdf/leg.urdf.xacro (robot description, xacro)
@@ -127,6 +127,6 @@
             <kp>1000000.0</kp>
             <kd>1.0</kd>
-            <mu1>0.8</mu1>
-            <mu2>0.8</mu2>
+            <mu1>1</mu1>
+            <mu2>1</mu2>
             <maxVel>0.0</maxVel>
             <minDepth>0.001</minDepth>
